Commit message: added colors

File: urdf/materials.xacro (robot description, xacro)
@@ -4,3 +4,6 @@
   <color rgba="0.700 0.700 0.700 1.000"/>
 </material>
+<material name="blue">
+  <color rgba="0.000 0.000 0.700 1.000"/>
+</material>
 </robot>

File: urdf/scuttle.xacro (robot description, xacro)
@@ -35,5 +35,5 @@
       <mesh filename="package://scuttle_description/meshes/l_wheel_1.stl" scale="0.001 0.001 0.001"/>
     </geometry>
-    <material name="silver"/>
+    <material name="blue"/>
   </visual>
   <collision>
@@ -55,5 +55,5 @@
       <mesh filename="package://scuttle_description/meshes/r_wheel_1.stl" scale="0.001 0.001 0.001"/>
     </geometry>
-    <material name="silver"/>
+    <material name="blue"/>
   </visual>
   <collision>
@@ -135,5 +135,5 @@
       <mesh filename="package://scuttle_description/meshes/l_caster_wheel_1.stl" scale="0.001 0.001 0.001"/>
     </geometry>
-    <material name="silver"/>
+    <material name="blue"/>
   </visual>
   <collision>
@@ -155,5 +155,5 @@
       <mesh filename="package://scuttle_description/meshes/r_caster_wheel_1.stl" scale="0.001 0.001 0.001"/>
     </geometry>
-    <material name="silver"/>
+    <material name="blue"/>
   </visual>
   <collision>

Commit message: added colors

File: urdf/materials.xacro (robot description, xacro)
@@ -4,4 +4,7 @@
   <color rgba="0.700 0.700 0.700 1.000"/>
 </material>
+<material name="gray">
+  <color rgba="0.250 0.250 0.250 1.000"/>
+</material>
 <material name="blue">
   <color rgba="0.000 0.000 0.700 1.000"/>

File: urdf/scuttle.xacro (robot description, xacro)
@@ -75,5 +75,5 @@
       <mesh filename="package://scuttle_description/meshes/LiDAR_1.stl" scale="0.001 0.001 0.001"/>
     </geometry>
-    <material name="silver"/>
+    <material name="gray"/>
   </visual>
   <collision>
