Commit message: fix lidar rotation

File: urdf/scuttle.xacro (robot description, xacro)
@@ -177,5 +177,5 @@
 </joint>
 <joint name="lidar" type="fixed">
-  <origin rpy="0 0 0" xyz="0.0 -0.0275 0.1096"/>
+  <origin rpy="0 0 1.570796" xyz="0.0 -0.0275 0.1096"/>
   <parent link="base_link"/>
   <child link="LiDAR_1"/>

Commit message: renamed lidar

File: urdf/scuttle.xacro (robot description, xacro)
@@ -64,5 +64,5 @@
   </collision>
 </link>
-<link name="LiDAR_1">
+<link name="lidar">
   <inertial>
     <origin rpy="0 0 0" xyz="-0.0010241190327231165 -0.0008953477993804172 0.009594767416774092"/>
@@ -73,5 +73,5 @@
     <origin rpy="0 0 0" xyz="-0.0 0.0275 -0.1096"/>
     <geometry>
-      <mesh filename="package://scuttle_description/meshes/LiDAR_1.stl" scale="0.001 0.001 0.001"/>
+      <mesh filename="package://scuttle_description/meshes/lidar.stl" scale="0.001 0.001 0.001"/>
     </geometry>
     <material name="gray"/>
@@ -80,5 +80,5 @@
     <origin rpy="0 0 0" xyz="-0.0 0.0275 -0.1096"/>
     <geometry>
-      <mesh filename="package://scuttle_description/meshes/LiDAR_1.stl" scale="0.001 0.001 0.001"/>
+      <mesh filename="package://scuttle_description/meshes/lidar.stl" scale="0.001 0.001 0.001"/>
     </geometry>
   </collision>
@@ -179,5 +179,5 @@
   <origin rpy="0 0 1.570796" xyz="0.0 -0.0275 0.1096"/>
   <parent link="base_link"/>
-  <child link="LiDAR_1"/>
+  <child link="lidar"/>
   <axis xyz="0.0 0.0 1.0"/>
 </joint>

Commit message: fixed lidar names

File: urdf/scuttle.xacro (robot description, xacro)
@@ -64,5 +64,5 @@
   </collision>
 </link>
-<link name="lidar">
+<link name="LiDAR_1">
   <inertial>
     <origin rpy="0 0 0" xyz="-0.0010241190327231165 -0.0008953477993804172 0.009594767416774092"/>
@@ -73,5 +73,5 @@
     <origin rpy="0 0 0" xyz="-0.0 0.0275 -0.1096"/>
     <geometry>
-      <mesh filename="package://scuttle_description/meshes/lidar.stl" scale="0.001 0.001 0.001"/>
+      <mesh filename="package://scuttle_description/meshes/LiDAR_1.stl" scale="0.001 0.001 0.001"/>
     </geometry>
     <material name="gray"/>
@@ -80,5 +80,5 @@
     <origin rpy="0 0 0" xyz="-0.0 0.0275 -0.1096"/>
     <geometry>
-      <mesh filename="package://scuttle_description/meshes/lidar.stl" scale="0.001 0.001 0.001"/>
+      <mesh filename="package://scuttle_description/meshes/LiDAR_1.stl" scale="0.001 0.001 0.001"/>
     </geometry>
   </collision>
@@ -179,5 +179,5 @@
   <origin rpy="0 0 1.570796" xyz="0.0 -0.0275 0.1096"/>
   <parent link="base_link"/>
-  <child link="lidar"/>
+  <child link="LiDAR_1"/>
   <axis xyz="0.0 0.0 1.0"/>
 </joint>

Commit message: fixed lidar error

File: urdf/scuttle.xacro (robot description, xacro)
@@ -6,7 +6,7 @@
 <link name="base_link">
   <inertial>
-    <origin rpy="0 0 0" xyz="2.12433370053547e-05 -0.07877992189559235 0.07392475478815927"/>
+    <origin rpy="0 0 0" xyz="2.12433370053547e-05 -0.07877992189559235 0.07392564365565002"/>
     <mass value="3.288323846275119"/>
-    <inertia ixx="0.038876" ixy="1.3e-05" ixz="2e-06" iyy="0.047513" iyz="0.000485" izz="0.084083"/>
+    <inertia ixx="0.038876" ixy="1.3e-05" ixz="1e-06" iyy="0.047513" iyz="0.000486" izz="0.084083"/>
   </inertial>
   <visual>
@@ -20,5 +20,5 @@
     <origin rpy="0 0 0" xyz="0 0 0"/>
     <geometry>
-      <mesh filename="package://scuttle_description/meshes/base_link_collision_1.stl" scale="0.001 0.001 0.001"/>
+      <mesh filename="package://scuttle_description/meshes/base_link.stl" scale="0.001 0.001 0.001"/>
     </geometry>
   </collision>
@@ -40,5 +40,5 @@
     <origin rpy="0 0 0" xyz="-0.21235 -0.0 -0.04175"/>
     <geometry>
-      <mesh filename="package://scuttle_description/meshes/l_wheel_collision_1.stl" scale="0.001 0.001 0.001"/>
+      <mesh filename="package://scuttle_description/meshes/l_wheel_1.stl" scale="0.001 0.001 0.001"/>
     </geometry>
   </collision>
@@ -60,9 +60,9 @@
     <origin rpy="0 0 0" xyz="0.21215 0.0 -0.04175"/>
     <geometry>
-      <mesh filename="package://scuttle_description/meshes/r_wheel_collision_1.stl" scale="0.001 0.001 0.001"/>
-    </geometry>
-  </collision>
-</link>
-<link name="LiDAR_1">
+      <mesh filename="package://scuttle_description/meshes/r_wheel_1.stl" scale="0.001 0.001 0.001"/>
+    </geometry>
+  </collision>
+</link>
+<link name="lidar_1">
   <inertial>
     <origin rpy="0 0 0" xyz="-0.0010241190327231165 -0.0008953477993804172 0.009594767416774092"/>
@@ -73,5 +73,5 @@
     <origin rpy="0 0 0" xyz="-0.0 0.0275 -0.1096"/>
     <geometry>
-      <mesh filename="package://scuttle_description/meshes/LiDAR_1.stl" scale="0.001 0.001 0.001"/>
+      <mesh filename="package://scuttle_description/meshes/lidar_1.stl" scale="0.001 0.001 0.001"/>
     </geometry>
     <material name="gray"/>
@@ -80,5 +80,5 @@
     <origin rpy="0 0 0" xyz="-0.0 0.0275 -0.1096"/>
     <geometry>
-      <mesh filename="package://scuttle_description/meshes/LiDAR_1.stl" scale="0.001 0.001 0.001"/>
+      <mesh filename="package://scuttle_description/meshes/lidar_1.stl" scale="0.001 0.001 0.001"/>
     </geometry>
   </collision>
@@ -100,5 +100,5 @@
     <origin rpy="0 0 0" xyz="0.119279 0.254415 -0.059282"/>
     <geometry>
-      <mesh filename="package://scuttle_description/meshes/r_caster_swivel_collision_1.stl" scale="0.001 0.001 0.001"/>
+      <mesh filename="package://scuttle_description/meshes/r_caster_swivel_1.stl" scale="0.001 0.001 0.001"/>
     </geometry>
   </collision>
@@ -120,5 +120,5 @@
     <origin rpy="0 0 0" xyz="-0.119015 0.254415 -0.059282"/>
     <geometry>
-      <mesh filename="package://scuttle_description/meshes/l_caster_swivel_collision_1.stl" scale="0.001 0.001 0.001"/>
+      <mesh filename="package://scuttle_description/meshes/l_caster_swivel_1.stl" scale="0.001 0.001 0.001"/>
     </geometry>
   </collision>
@@ -140,5 +140,5 @@
     <origin rpy="0 0 0" xyz="-0.101223 0.230415 -0.025282"/>
     <geometry>
-      <mesh filename="package://scuttle_description/meshes/l_caster_wheel_collision_1.stl" scale="0.001 0.001 0.001"/>
+      <mesh filename="package://scuttle_description/meshes/l_caster_wheel_1.stl" scale="0.001 0.001 0.001"/>
     </geometry>
   </collision>
@@ -160,5 +160,5 @@
     <origin rpy="0 0 0" xyz="0.105071 0.230415 -0.025282"/>
     <geometry>
-      <mesh filename="package://scuttle_description/meshes/r_caster_wheel_collision_1.stl" scale="0.001 0.001 0.001"/>
+      <mesh filename="package://scuttle_description/meshes/r_caster_wheel_1.stl" scale="0.001 0.001 0.001"/>
     </geometry>
   </collision>
@@ -177,8 +177,7 @@
 </joint>
 <joint name="lidar" type="fixed">
-  <origin rpy="0 0 1.570796" xyz="0.0 -0.0275 0.1096"/>
-  <parent link="base_link"/>
-  <child link="LiDAR_1"/>
-  <axis xyz="0.0 0.0 1.0"/>
+  <origin rpy="0 0 0" xyz="0.0 -0.0275 0.1096"/>
+  <parent link="base_link"/>
+  <child link="lidar_1"/>
 </joint>
 <joint name="r_caster_swivel_joint" type="continuous">

Commit message: fixed collision meshes

File: urdf/scuttle.xacro (robot description, xacro)
@@ -20,5 +20,5 @@
     <origin rpy="0 0 0" xyz="0 0 0"/>
     <geometry>
-      <mesh filename="package://scuttle_description/meshes/base_link.stl" scale="0.001 0.001 0.001"/>
+      <mesh filename="package://scuttle_description/meshes/base_link_collision_1.stl" scale="0.001 0.001 0.001"/>
     </geometry>
   </collision>
@@ -40,5 +40,5 @@
     <origin rpy="0 0 0" xyz="-0.21235 -0.0 -0.04175"/>
     <geometry>
-      <mesh filename="package://scuttle_description/meshes/l_wheel_1.stl" scale="0.001 0.001 0.001"/>
+      <mesh filename="package://scuttle_description/meshes/l_wheel_collision_1.stl" scale="0.001 0.001 0.001"/>
     </geometry>
   </collision>
@@ -60,5 +60,5 @@
     <origin rpy="0 0 0" xyz="0.21215 0.0 -0.04175"/>
     <geometry>
-      <mesh filename="package://scuttle_description/meshes/r_wheel_1.stl" scale="0.001 0.001 0.001"/>
+      <mesh filename="package://scuttle_description/meshes/r_wheel_collision_1.stl" scale="0.001 0.001 0.001"/>
     </geometry>
   </collision>
@@ -100,5 +100,5 @@
     <origin rpy="0 0 0" xyz="0.119279 0.254415 -0.059282"/>
     <geometry>
-      <mesh filename="package://scuttle_description/meshes/r_caster_swivel_1.stl" scale="0.001 0.001 0.001"/>
+      <mesh filename="package://scuttle_description/meshes/r_caster_swivel_collision_1.stl" scale="0.001 0.001 0.001"/>
     </geometry>
   </collision>
@@ -120,5 +120,5 @@
     <origin rpy="0 0 0" xyz="-0.119015 0.254415 -0.059282"/>
     <geometry>
-      <mesh filename="package://scuttle_description/meshes/l_caster_swivel_1.stl" scale="0.001 0.001 0.001"/>
+      <mesh filename="package://scuttle_description/meshes/l_caster_swivel_collision_1.stl" scale="0.001 0.001 0.001"/>
     </geometry>
   </collision>
@@ -140,5 +140,5 @@
     <origin rpy="0 0 0" xyz="-0.101223 0.230415 -0.025282"/>
     <geometry>
-      <mesh filename="package://scuttle_description/meshes/l_caster_wheel_1.stl" scale="0.001 0.001 0.001"/>
+      <mesh filename="package://scuttle_description/meshes/l_caster_wheel_collision_1.stl" scale="0.001 0.001 0.001"/>
     </geometry>
   </collision>
@@ -160,5 +160,5 @@
     <origin rpy="0 0 0" xyz="0.105071 0.230415 -0.025282"/>
     <geometry>
-      <mesh filename="package://scuttle_description/meshes/r_caster_wheel_1.stl" scale="0.001 0.001 0.001"/>
+      <mesh filename="package://scuttle_description/meshes/r_caster_wheel_collision_1.stl" scale="0.001 0.001 0.001"/>
     </geometry>
   </collision>

Commit message: fixed lidar rotation

File: urdf/scuttle.xacro (robot description, xacro)
@@ -177,5 +177,5 @@
 </joint>
 <joint name="lidar" type="fixed">
-  <origin rpy="0 0 0" xyz="0.0 -0.0275 0.1096"/>
+  <origin rpy="0 0 1.570796" xyz="0.0 -0.0275 0.1096"/>
   <parent link="base_link"/>
   <child link="lidar_1"/>

Commit message: fixed SCUTTLE coordinate frame

File: urdf/scuttle.xacro (robot description, xacro)
@@ -11,5 +11,5 @@
   </inertial>
   <visual>
-    <origin rpy="0 0 0" xyz="0 0 0"/>
+    <origin rpy="0 0 1.570796" xyz="0 0 0"/>
     <geometry>
       <mesh filename="package://scuttle_description/meshes/base_link.stl" scale="0.001 0.001 0.001"/>
@@ -165,5 +165,5 @@
 </link>
 <joint name="l_wheel_joint" type="continuous">
-  <origin rpy="0 0 0" xyz="0.21235 0.0 0.04175"/>
+  <origin rpy="0 0 1.570796" xyz="0.0 0.21235 0.04175"/>
   <parent link="base_link"/>
   <child link="l_wheel_1"/>
@@ -171,5 +171,5 @@
 </joint>
 <joint name="r_wheel_joint" type="continuous">
-  <origin rpy="0 0 0" xyz="-0.21215 0.0 0.04175"/>
+  <origin rpy="0 0 1.570796" xyz="0.0 -0.21215 0.04175"/>
   <parent link="base_link"/>
   <child link="r_wheel_1"/>
@@ -177,10 +177,10 @@
 </joint>
 <joint name="lidar" type="fixed">
-  <origin rpy="0 0 1.570796" xyz="0.0 -0.0275 0.1096"/>
+  <origin rpy="0 0 0" xyz="0.0275 0.0 0.1096"/>
   <parent link="base_link"/>
   <child link="lidar_1"/>
 </joint>
 <joint name="r_caster_swivel_joint" type="continuous">
-  <origin rpy="0 0 0" xyz="-0.119279 -0.254415 0.059282"/>
+  <origin rpy="0 0 1.570796" xyz="0.254415 0.119279 0.059282"/>
   <parent link="base_link"/>
   <child link="r_caster_swivel_1"/>
@@ -188,5 +188,5 @@
 </joint>
 <joint name="l_caster_swivel_joint" type="continuous">
-  <origin rpy="0 0 0" xyz="0.119015 -0.254415 0.059282"/>
+  <origin rpy="0 0 1.570796" xyz="0.254415 -0.119015 0.059282"/>
   <parent link="base_link"/>
   <child link="l_caster_swivel_1"/>

Commit message: fixed lidar rotation with new coordinate frame

File: urdf/scuttle.xacro (robot description, xacro)
@@ -177,5 +177,5 @@
 </joint>
 <joint name="lidar" type="fixed">
-  <origin rpy="0 0 0" xyz="0.0275 0.0 0.1096"/>
+  <origin rpy="0 0 3.141592" xyz="0.0275 0.0 0.1096"/>
   <parent link="base_link"/>
   <child link="lidar_1"/>

Commit message: Update scuttle.xacro

File: urdf/scuttle.xacro (robot description, xacro)
@@ -18,5 +18,5 @@
   </visual>
   <collision>
-    <origin rpy="0 0 0" xyz="0 0 0"/>
+    <origin rpy="0 0 1.570796" xyz="0 0 0"/>
     <geometry>
       <mesh filename="package://scuttle_description/meshes/base_link_collision_1.stl" scale="0.001 0.001 0.001"/>

Commit message: Attempted fix for SCUTTLE base_link inertia

File: urdf/scuttle.xacro (robot description, xacro)
@@ -6,5 +6,5 @@
 <link name="base_link">
   <inertial>
-    <origin rpy="0 0 0" xyz="2.12433370053547e-05 -0.07877992189559235 0.07392564365565002"/>
+    <origin rpy="0 0 0" xyz="0.1 0 0.07392564365565002"/>
     <mass value="3.288323846275119"/>
     <inertia ixx="0.038876" ixy="1.3e-05" ixz="1e-06" iyy="0.047513" iyz="0.000486" izz="0.084083"/>
